File: mcu.kicad_sch (KiCad schematic)
At the start: 15 parts, among them U1 STM32F405RGTx, Y1 8MHz

Commit message: more stuff
Parts:
- R14, R15: value 1k -> 22k
Connections:
- net MCU_VBAT: now reaches U1.1 (VBAT)
Other:
- moved on the sheet: C10, C11, C14, C15, C7, C8, C9, FB2, FB3, Y1

Commit message: imported SA868 - thanks, edgetriggered
Parts:
- added C3: 100n, Capacitor_SMD:C_0805_2012Metric, symbol Device:C
- renumbered C13 to C1, C11 to C10, C12 to C2, C15 to C4, C14 to C5, C7 to C6, C8 to C7, C9 to C8, C10 to C9, FB2 to FB1, FB3 to FB2, R15 to R1, R14 to R2
Connections:
- net GND: now also C3.1
- net MCU_VBAT renamed RTC_BATT
- net RTC_BATT: now also C3.2

Commit message: interfaces update
Connections:
- net UDB_DM: now also U1.44 (PA11)
- net USB_DP: now also U1.45 (PA12)
Changed lines of the file:
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@@
 	(title_block
 		(title "Mainboard replacement for Nokia 3310")
-		(date "23-10-2024")
+		(date "24-10-2024")
 		(rev "Rev A")
 		(company "M17 Project")
@@
 	(wire
 		(pts
+			(xy 165.1 85.09) (xy 161.29 85.09)
+		)
+		(stroke
+			(width 0)
+			(type default)
+		)
+	)
+	(wire
+		(pts
 			(xy 121.92 67.31) (xy 125.73 67.31)
 		)
@@
 		)
 	)
+	(bus
+		(pts
+			(xy 190.5 100.33) (xy 212.09 100.33)
+		)
+		(stroke
+			(width 0)
+			(type default)
+		)
+	)
 	(wire
 		(pts
@@
 	(wire
 		(pts
+			(xy 165.1 87.63) (xy 161.29 87.63)
+		)
+		(stroke
+			(width 0)
+			(type default)
+		)
+	)
+	(wire
+		(pts
 			(xy 265.43 40.64) (xy 267.97 40.64)
 		)
@@
 		(pts
 			(xy 143.51 146.05) (xy 143.51 148.59)
+		)
+		(stroke
+			(width 0)
+			(type default)
+		)
+	)
+	(bus
+		(pts
+			(xy 190.5 97.79) (xy 212.09 97.79)
 		)
 		(stroke
@@
 		)
 	)
+	(label "{KEY_ROWS}"
+		(at 191.77 97.79 0)
+		(fields_autoplaced yes)
+		(effects
+			(font
+				(size 1.27 1.27)
+			)
+			(justify left bottom)
+		)
+	)
+	(label "{KEY_COLS}"
+		(at 191.77 100.33 0)
+		(fields_autoplaced yes)
+		(effects
+			(font
+				(size 1.27 1.27)
+			)
+			(justify left bottom)
+		)
+	)
+	(hierarchical_label "KEY_COLS"
+		(shape output)
+		(at 212.09 100.33 0)
+		(fields_autoplaced yes)
+		(effects
+			(font
+				(size 1.27 1.27)
+			)
+			(justify left)
+		)
+	)
 	(hierarchical_label "UDB_DM"
 		(shape bidirectional)
-		(at 212.09 100.33 0)
+		(at 165.1 85.09 0)
 		(fields_autoplaced yes)
 		(effects
@@
 	(hierarchical_label "USB_DP"
 		(shape bidirectional)
-		(at 212.09 97.79 0)
+		(at 165.1 87.63 0)
 		(fields_autoplaced yes)
 		(effects
@@
 			)
 			(justify left)
+		)
+	)
+	(hierarchical_label "DISP_DATA"
+		(shape output)
+		(at 104.14 91.44 180)
+		(fields_autoplaced yes)
+		(effects
+			(font
+				(size 1.27 1.27)
+			)
+			(justify right)
 		)
 	)
@@
 		)
 	)
+	(hierarchical_label "PTT_OUT"
+		(shape output)
+		(at 104.14 78.74 180)
+		(fields_autoplaced yes)
+		(effects
+			(font
+				(size 1.27 1.27)
+			)
+			(justify right)
+		)
+	)
+	(hierarchical_label "~{DISP_CE}"
+		(shape output)
+		(at 104.14 99.06 180)
+		(fields_autoplaced yes)
+		(effects
+			(font
+				(size 1.27 1.27)
+			)
+			(justify right)
+		)
+	)
+	(hierarchical_label "RF_PWR"
+		(shape output)
+		(at 104.14 83.82 180)
+		(fields_autoplaced yes)
+		(effects
+			(font
+				(size 1.27 1.27)
+			)
+			(justify right)
+		)
+	)
 	(hierarchical_label "RF_RX"
 		(shape input)
@@
 		)
 	)
+	(hierarchical_label "DISP_D{slash}C"
+		(shape output)
+		(at 104.14 93.98 180)
+		(fields_autoplaced yes)
+		(effects
+			(font
+				(size 1.27 1.27)
+			)
+			(justify right)
+		)
+	)
+	(hierarchical_label "RF_ENA"
+		(shape output)
+		(at 104.14 81.28 180)
+		(fields_autoplaced yes)
+		(effects
+			(font
+				(size 1.27 1.27)
+			)
+			(justify right)
+		)
+	)
+	(hierarchical_label "KEY_ROWS"
+		(shape input)
+		(at 212.09 97.79 0)
+		(fields_autoplaced yes)
+		(effects
+			(font
+				(size 1.27 1.27)
+			)
+			(justify left)
+		)
+	)
 	(hierarchical_label "RF_TX"
 		(shape output)
@@
 		)
 	)
+	(hierarchical_label "~{DISP_RST}"
+		(shape output)
+		(at 104.14 96.52 180)
+		(fields_autoplaced yes)
+		(effects
+			(font
+				(size 1.27 1.27)
+			)
+			(justify right)
+		)
+	)
+	(hierarchical_label "PWM_BLIGHT"
+		(shape output)
+		(at 104.14 86.36 180)
+		(fields_autoplaced yes)
+		(effects
+			(font
+				(size 1.27 1.27)
+			)
+			(justify right)
+		)
+	)
+	(hierarchical_label "DISP_SCK"
+		(shape output)
+		(at 104.14 88.9 180)
+		(fields_autoplaced yes)
+		(effects
+			(font
+				(size 1.27 1.27)
+			)
+			(justify right)
+		)
+	)

Commit message: connections
Parts:
- added D1: 3V3, symbol Device:D_Zener
- added J1: SWD_DBG, symbol Connector:Conn_01x04_Pin
- added R2: 2k2, Inductor_SMD:L_0805_2012Metric, symbol Device:R
- added R3, R5: 10k, Inductor_SMD:L_0805_2012Metric, symbol Device:R
- added R6: 1k, Inductor_SMD:L_0805_2012Metric, symbol Device:R
- renumbered C4 to C1, C5 to C2, C1 to C3, C2 to C4, C3 to C5, R2 to R4
Connections:
- net +3V3: now also R3.1, R5.1
- net DISP_DATA: now also U1.57 (PB5)
- net DISP_D/C: now also U1.59 (PB7)
- net DISP_SCK: now also U1.55 (PB3)
- net GND: now also D1.2 (A), J1.4 (Pin_4)
- net MCU_VDD: now also R2.1
- net RF_RX: now also R6.1
- net ~{DISP_CE}: now also U1.58 (PB6)
- net ~{DISP_RST}: now also U1.61 (PB8)
- net BSB_IN: now reaches U1.14 (PA0)
- net MIC_IN: now reaches U1.15 (PA1)
- net BSB_OUT: now reaches U1.20 (PA4)
- net SPK_OUT: now reaches U1.21 (PA5)
- net ~{CHG}: now reaches U1.35 (PB14)
- net ~{CHG}: now also R5.2
- net PWR_ON: now reaches U1.36 (PB15)
- net SD_D0: now reaches U1.39 (PC8)
- net SD_D1: now reaches U1.40 (PC9)
- net SWDIO: now reaches U1.46 (PA13)
- net SWDIO: now also J1.2 (Pin_2)
- net SWCLK: now reaches U1.49 (PA14)
- net SWCLK: now also J1.3 (Pin_3)
- net SD_DET: now reaches U1.50 (PA15)
- net SD_DET: now also R3.2
- net SD_D2: now reaches U1.51 (PC10)
- net SD_D3: now reaches U1.52 (PC11)
- net SD_CLK: now reaches U1.53 (PC12)
- net SD_CMD: now reaches U1.54 (PD2)
- net NRST: now reaches U1.7 (NRST)
- net NRST: now also J1.1 (Pin_1), R2.2
- new net: D1.1 (K), R6.2
- no-connect marks 0 -> 1
Other:
- moved on the sheet: C1, C2, R4, Y1
