File: mcu.kicad_sch (KiCad schematic)
At the start: 21 parts, among them J1 SWD_DBG, U1 STM32F405RGTx, Y1 8MHz

Commit message: more pcb routing
Parts:
- renumbered R6 to R5, R5 to R6
Connections:
- net +3V3: no longer R5.1
- net MCU_VDD: now also R5.1
- net ~{CHG}: now also U1.21 (PA5); no longer U1.35 (PB14)
- net 32k_X1: no longer names the net of U1.3 (PC14)
- net 32k_X2: no longer names the net of U1.4 (PC15)
- net PWR_ON renamed PWR_OFF
- no-connect marks 1 -> 3
Other:
- moved on the sheet: R5
Changed lines of the file:
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@@
 	(title_block
 		(title "Mainboard replacement for Nokia 3310")
-		(date "2-11-2024")
+		(date "3-11-2024")
 		(rev "Rev A")
 		(company "M17 Project")
@@
 	)
 	(junction
-		(at 173.99 135.89)
-		(diameter 0)
-		(color 0 0 0 0)
-	)
-	(junction
 		(at 146.05 49.53)
 		(diameter 0)
@@
 	)
 	(junction
+		(at 163.83 69.85)
+		(diameter 0)
+		(color 0 0 0 0)
+	)
+	(junction
 		(at 265.43 40.64)
 		(diameter 0)
@@
 		(at 161.29 110.49)
 	)
+	(no_connect
+		(at 125.73 118.11)
+	)
+	(no_connect
+		(at 125.73 115.57)
+	)
 	(bus_entry
 		(at 254 123.19)
@@
 	(wire
 		(pts
-			(xy 180.34 133.35) (xy 173.99 133.35)
+			(xy 161.29 69.85) (xy 163.83 69.85)
+		)
+		(stroke
+			(width 0)
+			(type default)
+		)
+	)
+	(wire
+		(pts
+			(xy 177.8 72.39) (xy 163.83 72.39)
 		)
 		(stroke
@@
 	(wire
 		(pts
-			(xy 173.99 133.35) (xy 173.99 135.89)
+			(xy 163.83 72.39) (xy 163.83 69.85)
 		)
 		(stroke
@@
 	(wire
 		(pts
-			(xy 161.29 135.89) (xy 173.99 135.89)
-		)
-		(stroke
-			(width 0)
-			(type default)
-		)
-	)
-	(wire
-		(pts
 			(xy 107.95 62.23) (xy 107.95 64.77)
 		)
@@
 	(wire
 		(pts
-			(xy 175.26 135.89) (xy 173.99 135.89)
+			(xy 165.1 69.85) (xy 163.83 69.85)
 		)
 		(stroke
@@
 	(wire
 		(pts
-			(xy 111.76 115.57) (xy 125.73 115.57)
-		)
-		(stroke
-			(width 0)
-			(type default)
-		)
-	)
-	(wire
-		(pts
-			(xy 190.5 133.35) (xy 187.96 133.35)
+			(xy 187.96 72.39) (xy 185.42 72.39)
 		)
 		(stroke
@@
 	(wire
 		(pts
-			(xy 190.5 132.08) (xy 190.5 133.35)
-		)
-		(stroke
-			(width 0)
-			(type default)
-		)
-	)
-	(wire
-		(pts
 			(xy 53.34 38.1) (xy 55.88 38.1)
 		)
@@
 	(wire
 		(pts
-			(xy 111.76 118.11) (xy 125.73 118.11)
-		)
-		(stroke
-			(width 0)
-			(type default)
-		)
-	)
-	(wire
-		(pts
 			(xy 161.29 49.53) (xy 163.83 49.53)
 		)
@@
 	)
 	(label "MCU_VDD"
-		(at 118.11 38.1 90)
+		(at 118.11 38.1 180)
 		(fields_autoplaced yes)
 		(effects
@@
 				(size 1.27 1.27)
 			)
-			(justify left bottom)
+			(justify right bottom)
 		)
 	)
@@
 		)
 	)
-	(label "32k_X1"
-		(at 111.76 115.57 180)
-		(fields_autoplaced yes)
-		(effects
-			(font
-				(size 1.27 1.27)
-			)
-			(justify right bottom)
-		)
-	)
-	(label "32k_X2"
-		(at 111.76 118.11 180)
+	(label "X2"
+		(at 121.92 69.85 180)
 		(fields_autoplaced yes)
 		(effects
@@
 		)
 	)
-	(label "X2"
-		(at 121.92 69.85 180)
+	(label "MCU_VDD"
+		(at 187.96 72.39 0)
 		(fields_autoplaced yes)
 		(effects
@@
 				(size 1.27 1.27)
 			)
-			(justify right bottom)
+			(justify left bottom)
 		)
 	)
@@
 		)
 	)
-	(hierarchical_label "PWR_ON"
+	(hierarchical_label "PWR_OFF"
 		(shape output)
 		(at 165.1 138.43 0)
@@
 	(hierarchical_label "~{CHG}"
 		(shape input)
-		(at 175.26 135.89 0)
+		(at 165.1 69.85 0)
 		(fields_autoplaced yes)
 		(effects
@@
 	(symbol
 		(lib_id "Device:R")
-		(at 184.15 133.35 270)
+		(at 181.61 72.39 270)
 		(unit 1)
 		(exclude_from_sim no)
@@
 		(on_board yes)
 		(dnp no)
-		(property "Reference" "R6"
-			(at 184.15 130.81 90)
+		(property "Reference" "R5"
+			(at 181.61 69.85 90)
 			(effects
 				(font
@@
 		)
 		(property "Value" "10k"
-			(at 184.15 135.89 90)
+			(at 181.61 74.93 90)
 			(effects
 				(font
@@
 		)
 		(property "Footprint" "Resistor_SMD:R_0402_1005Metric"
-			(at 184.15 131.572 90)
+			(at 181.61 70.612 90)
 			(effects
 				(font
@@
 		)
 		(property "Datasheet" "~"
-			(at 184.15 133.35 0)
+			(at 181.61 72.39 0)
 			(effects
 				(font
@@
 		)
 		(property "Description" "Resistor"
-			(at 184.15 133.35 0)
+			(at 181.61 72.39 0)
 			(effects
 				(font
@@
 		)
 		(property "PN" ""
-			(at 184.15 133.35 0)
+			(at 181.61 72.39 0)
 			(effects
 				(font
@@
 		)
 		(property "MPN" ""
-			(at 184.15 133.35 0)
+			(at 181.61 72.39 0)
 			(effects
 				(font
@@
 			(project "M17_3310"
 				(path "/8d65c5ef-7a02-4454-aee5-ab9c49e4aeab/d70e0f3c-6f62-45eb-a17e-0f32c3e4716f"
-					(reference "R6")
+					(reference "R5")
 					(unit 1)
 				)
@@
 		(dnp no)
 		(fields_autoplaced yes)
-		(property "Reference" "#PWR023"
+		(property "Reference" "#PWR022"
 			(at 231.14 57.15 0)
 			(effects
@@
 			(project "M17_3310"
 				(path "/8d65c5ef-7a02-4454-aee5-ab9c49e4aeab/d70e0f3c-6f62-45eb-a17e-0f32c3e4716f"
-					(reference "#PWR023")
+					(reference "#PWR022")
 					(unit 1)
 				)
@@
 		(dnp no)
 		(fields_autoplaced yes)
-		(property "Reference" "#PWR024"
+		(property "Reference" "#PWR023"
 			(at 242.57 57.15 0)
 			(effects
@@
 			(project "M17_3310"
 				(path "/8d65c5ef-7a02-4454-aee5-ab9c49e4aeab/d70e0f3c-6f62-45eb-a17e-0f32c3e4716f"
-					(reference "#PWR024")
-					(unit 1)
-				)
-			)
-		)
-	)
-	(symbol
-		(lib_id "power:+3V3")
-		(at 190.5 132.08 0)
-		(unit 1)
-		(exclude_from_sim no)
-		(in_bom yes)
-		(on_board yes)
-		(dnp no)
-		(fields_autoplaced yes)
-		(property "Reference" "#PWR020"
-			(at 190.5 135.89 0)
-			(effects
-				(font
-					(size 1.27 1.27)
-				)
-				(hide yes)
-			)
-		)
-		(property "Value" "+3V3"
-			(at 190.5 127 0)
-			(effects
-				(font
-					(size 1.27 1.27)
-				)
-			)
-		)
-		(property "Footprint" ""
-			(at 190.5 132.08 0)
-			(effects
-				(font
-					(size 1.27 1.27)
-				)
-				(hide yes)
-			)
-		)
-		(property "Datasheet" ""
-			(at 190.5 132.08 0)
-			(effects
-				(font
-					(size 1.27 1.27)
-				)
-				(hide yes)
-			)
-		)
-		(property "Description" "Power symbol creates a global label with name \"+3V3\""
-			(at 190.5 132.08 0)
-			(effects
-				(font
-					(size 1.27 1.27)
-				)
-				(hide yes)
-			)
-		)
-		(pin "1"
-		)
-		(instances
-			(project "M17_3310"
-				(path "/8d65c5ef-7a02-4454-aee5-ab9c49e4aeab/d70e0f3c-6f62-45eb-a17e-0f32c3e4716f"
-					(reference "#PWR020")
+					(reference "#PWR023")
 					(unit 1)
 				)
@@
 		(dnp no)
 		(fields_autoplaced yes)
-		(property "Reference" "#PWR022"
+		(property "Reference" "#PWR021"
 			(at 219.71 57.15 0)
 			(effects
@@
 			(project "M17_3310"
 				(path "/8d65c5ef-7a02-4454-aee5-ab9c49e4aeab/d70e0f3c-6f62-45eb-a17e-0f32c3e4716f"
-					(reference "#PWR022")
+					(reference "#PWR021")
 					(unit 1)
 				)
@@
 		(dnp no)
 		(fields_autoplaced yes)
-		(property "Reference" "#PWR021"
+		(property "Reference" "#PWR020"
 			(at 219.71 30.48 0)
 			(effects
@@
 			(project ""
 				(path "/8d65c5ef-7a02-4454-aee5-ab9c49e4aeab/d70e0f3c-6f62-45eb-a17e-0f32c3e4716f"
-					(reference "#PWR021")
+					(reference "#PWR020")
 					(unit 1)
 				)
@@
 		(dnp no)
 		(fields_autoplaced yes)
-		(property "Reference" "#PWR026"
+		(property "Reference" "#PWR025"
 			(at 265.43 57.15 0)
 			(effects
@@
 			(project "M17_3310"
 				(path "/8d65c5ef-7a02-4454-aee5-ab9c49e4aeab/d70e0f3c-6f62-45eb-a17e-0f32c3e4716f"
-					(reference "#PWR026")
+					(reference "#PWR025")
 					(unit 1)
 				)
@@
 		(dnp no)
 		(fields_autoplaced yes)
-		(property "Reference" "#PWR025"
+		(property "Reference" "#PWR024"
 			(at 254 57.15 0)
 			(effects
@@
 			(project "M17_3310"
 				(path "/8d65c5ef-7a02-4454-aee5-ab9c49e4aeab/d70e0f3c-6f62-45eb-a17e-0f32c3e4716f"
-					(reference "#PWR025")
+					(reference "#PWR024")
 					(unit 1)
 				)
@@
 		(on_board yes)
 		(dnp no)
-		(property "Reference" "R5"
+		(property "Reference" "R6"
 			(at 181.61 102.87 90)
 			(effects
@@
 			(project "M17_3310"
 				(path "/8d65c5ef-7a02-4454-aee5-ab9c49e4aeab/d70e0f3c-6f62-45eb-a17e-0f32c3e4716f"
-					(reference "R5")
+					(reference "R6")
 					(unit 1)
 				)

Commit message: more pcb routing
Parts:
- added Y2: 32.768kHz, Parts:xtal_smd_32k, symbol Device:Crystal
Connections:
- net COL_1: now also U1.33 (PB12)
- net COL_2: now also U1.11 (PC3)
- net COL_3: now also U1.9 (PC1)
- net ROW_1: now also U1.43 (PA10)
- net ROW_2: now also U1.42 (PA9)
- net ROW_3: now also U1.41 (PA8)
- net ROW_4: now also U1.40 (PC9)
- net ROW_5: now also U1.39 (PC8)
- net X1_32k: now reaches U1.3 (PC14)
- net X1_32k: now also Y2.1
- net X2_32k: now reaches U1.4 (PC15)
- net X2_32k: now also Y2.2
- no-connect marks 3 -> 1
