File: ifaces.kicad_sch (KiCad schematic)
At the start: 63 parts, among them J5 Vibrator, J6 Buzzer, J7 Display, J8 USB C, Q6 BSS138, Q7 BSS138, Q8 IRLML6401, Q9 BSS138, SW2 "OK", U5 USBLC6-2SC6

Commit message: USB C receptacle's PN update
Parts:
- J8: MPN 656-DX07S016JA1R1500 -> 640-USB4110-GF-A; PN 656-DX07S016JA1R1500 -> 640-USB4110-GF-A
Changed lines of the file:
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@@
 			)
 		)
-		(property "PN" "656-DX07S016JA1R1500"
+		(property "PN" "640-USB4110-GF-A"
 			(at 269.24 43.18 0)
 			(effects
@@
 			)
 		)
-		(property "MPN" "656-DX07S016JA1R1500"
+		(property "MPN" "640-USB4110-GF-A"
 			(at 269.24 43.18 0)
 			(effects

Commit message: some pcb updates
- linked vibrator/buzzer footprints
Parts:
- J5: footprint (none) -> Parts:3310_vibrator
- J6: footprint (none) -> Parts:3310_buzzer
Changed lines of the file:
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@@
 			)
 		)
-		(property "Footprint" ""
+		(property "Footprint" "Parts:3310_vibrator"
 			(at 35.56 88.9 0)
 			(effects
@@
 			)
 		)
-		(property "Footprint" ""
+		(property "Footprint" "Parts:3310_buzzer"
 			(at 69.85 88.9 0)
 			(effects

Commit message: pcb update
Parts:
- D10, D11, D12, D13, D5, D6, D7, D9: value LED -> RED; footprint (none) -> Parts:3310_led; MPN (none) -> 743-IN-S124ARUR; PN (none) -> 743-IN-S124ARUR
- R17, R18, R19, R20, R22, R30, R31, R32, R33, R34, R35, R36, R37: footprint Inductor_SMD:L_0805_2012Metric -> Resistor_SMD:R_0805_2012Metric
- R21, R23, R24, R25, R26, R27, R28, R29: value 27R -> 56R; footprint Inductor_SMD:L_0805_2012Metric -> Resistor_SMD:R_0805_2012Metric

Commit message: more pcb routing
Parts:
- C19, C20: footprint Capacitor_SMD:C_0805_2012Metric -> Capacitor_SMD:C_0402_1005Metric
- R17, R19, R20, R21, R22, R23, R24, R25, R26, R27, R28, R29, R30, R31, R32, R33, R34, R35, R36, R37: footprint Resistor_SMD:R_0805_2012Metric -> Resistor_SMD:R_0402_1005Metric
- R18: value 47R -> 56R; footprint Resistor_SMD:R_0805_2012Metric -> Resistor_SMD:R_0402_1005Metric
- SW16: footprint Parts:3310_key -> Parts:3310_key_gap
Connections:
- net UDB_DM: now also U5.3 (I/O2); no longer U5.1 (I/O1)
- net USB_DP: now also U5.1 (I/O1); no longer U5.3 (I/O2)
- net at J8.A6 (D+), J8.B6 (D+): now also U5.6 (I/O1); no longer U5.4 (I/O2)
- net at J8.A7 (D-), J8.B7 (D-): now also U5.4 (I/O2); no longer U5.6 (I/O1)
Changed lines of the file:
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@@
 	)
 	(junction
+		(at 251.46 45.72)
+		(diameter 0)
+		(color 0 0 0 0)
+	)
+	(junction
 		(at 212.09 113.03)
 		(diameter 0)
@@
 	)
 	(junction
-		(at 114.3 182.88)
+		(at 251.46 43.18)
 		(diameter 0)
 		(color 0 0 0 0)
 	)
 	(junction
-		(at 254 107.95)
+		(at 114.3 182.88)
 		(diameter 0)
 		(color 0 0 0 0)
 	)
 	(junction
-		(at 251.46 45.72)
+		(at 254 107.95)
 		(diameter 0)
 		(color 0 0 0 0)
@@
 	)
 	(junction
-		(at 251.46 43.18)
-		(diameter 0)
-		(color 0 0 0 0)
-	)
-	(junction
 		(at 229.87 97.79)
 		(diameter 0)
@@
 	(wire
 		(pts
-			(xy 223.52 43.18) (xy 226.06 43.18)
-		)
-		(stroke
-			(width 0)
-			(type default)
-		)
-	)
-	(wire
-		(pts
 			(xy 68.58 111.76) (xy 68.58 113.03)
 		)
@@
 	(wire
 		(pts
+			(xy 248.92 43.18) (xy 251.46 45.72)
+		)
+		(stroke
+			(width 0)
+			(type default)
+		)
+	)
+	(wire
+		(pts
 			(xy 231.14 27.94) (xy 231.14 38.1)
 		)
@@
 	(wire
 		(pts
+			(xy 223.52 43.18) (xy 226.06 43.18)
+		)
+		(stroke
+			(width 0)
+			(type default)
+		)
+	)
+	(wire
+		(pts
 			(xy 77.47 88.9) (xy 77.47 85.09)
 		)
@@
 	(wire
 		(pts
-			(xy 224.79 143.51) (xy 224.79 148.59)
+			(xy 223.52 45.72) (xy 226.06 45.72)
 		)
 		(stroke
@@
 	(wire
 		(pts
-			(xy 217.17 128.27) (xy 229.87 128.27)
+			(xy 224.79 143.51) (xy 224.79 148.59)
 		)
 		(stroke
@@
 	(wire
 		(pts
-			(xy 87.63 170.18) (xy 87.63 172.72)
+			(xy 217.17 128.27) (xy 229.87 128.27)
 		)
 		(stroke
@@
 	(wire
 		(pts
-			(xy 229.87 138.43) (xy 242.57 138.43)
+			(xy 87.63 170.18) (xy 87.63 172.72)
 		)
 		(stroke
@@
 	(wire
 		(pts
-			(xy 254 96.52) (xy 254 97.79)
+			(xy 229.87 138.43) (xy 242.57 138.43)
 		)
 		(stroke
@@
 	(wire
 		(pts
-			(xy 251.46 45.72) (xy 254 45.72)
+			(xy 254 96.52) (xy 254 97.79)
 		)
 		(stroke
@@
 	(wire
 		(pts
-			(xy 105.41 170.18) (xy 105.41 172.72)
+			(xy 251.46 45.72) (xy 254 45.72)
 		)
 		(stroke
@@
 	(wire
 		(pts
-			(xy 223.52 45.72) (xy 226.06 45.72)
+			(xy 105.41 170.18) (xy 105.41 172.72)
 		)
 		(stroke
@@
 	(wire
 		(pts
-			(xy 236.22 45.72) (xy 251.46 45.72)
-		)
-		(stroke
-			(width 0)
-			(type default)
-		)
-	)
-	(wire
-		(pts
 			(xy 254 97.79) (xy 260.35 97.79)
 		)
@@
 	(wire
 		(pts
+			(xy 251.46 43.18) (xy 248.92 45.72)
+		)
+		(stroke
+			(width 0)
+			(type default)
+		)
+	)
+	(wire
+		(pts
 			(xy 254 118.11) (xy 260.35 118.11)
 		)
@@
 	(wire
 		(pts
+			(xy 236.22 45.72) (xy 248.92 45.72)
+		)
+		(stroke
+			(width 0)
+			(type default)
+		)
+	)
+	(wire
+		(pts
 			(xy 96.52 161.29) (xy 105.41 161.29)
 		)
@@
 	(wire
 		(pts
-			(xy 236.22 43.18) (xy 251.46 43.18)
+			(xy 267.97 118.11) (xy 270.51 118.11)
 		)
 		(stroke
@@
 		)
 	)
-	(wire
+	(bus
 		(pts
-			(xy 267.97 118.11) (xy 270.51 118.11)
+			(xy 234.95 90.17) (xy 251.46 90.17)
 		)
 		(stroke
@@
 		)
 	)
-	(bus
+	(wire
 		(pts
-			(xy 234.95 90.17) (xy 251.46 90.17)
+			(xy 114.3 182.88) (xy 123.19 182.88)
 		)
 		(stroke
@@
 	(wire
 		(pts
-			(xy 114.3 182.88) (xy 123.19 182.88)
+			(xy 43.18 85.09) (xy 50.8 85.09)
 		)
 		(stroke
@@
 	(wire
 		(pts
-			(xy 43.18 85.09) (xy 50.8 85.09)
+			(xy 236.22 43.18) (xy 248.92 43.18)
 		)
 		(stroke
@@
 	(hierarchical_label "USB_DP"
 		(shape bidirectional)
-		(at 223.52 45.72 180)
+		(at 223.52 43.18 180)
 		(fields_autoplaced yes)
 		(effects
@@
 	(hierarchical_label "UDB_DM"
 		(shape bidirectional)
-		(at 223.52 43.18 180)
+		(at 223.52 45.72 180)
 		(fields_autoplaced yes)
 		(effects
@@
 			)
 		)
-		(property "Value" "47R"
+		(property "Value" "56R"
 			(at 38.1 167.64 90)
 			(effects
@@
 			)
 		)
-		(property "Footprint" "Resistor_SMD:R_0805_2012Metric"
+		(property "Footprint" "Resistor_SMD:R_0402_1005Metric"
 			(at 38.1 173.228 90)
 			(effects
@@
 			)
 		)
-		(property "Footprint" "Resistor_SMD:R_0805_2012Metric"
+		(property "Footprint" "Resistor_SMD:R_0402_1005Metric"
 			(at 76.962 166.37 90)
 			(effects
@@
 			)
 		)
-		(property "Footprint" "Resistor_SMD:R_0805_2012Metric"
+		(property "Footprint" "Resistor_SMD:R_0402_1005Metric"
 			(at 264.16 96.012 90)
 			(effects
@@
 			)
 		)
-		(property "Footprint" "Resistor_SMD:R_0805_2012Metric"
+		(property "Footprint" "Resistor_SMD:R_0402_1005Metric"
 			(at 94.742 166.37 90)
 			(effects
@@
 			)
 		)
-		(property "Footprint" "Resistor_SMD:R_0805_2012Metric"
+		(property "Footprint" "Resistor_SMD:R_0402_1005Metric"
 			(at 245.872 52.07 90)
 			(effects
@@
 			)
 		)
-		(property "Footprint" "Parts:3310_key"
+		(property "Footprint" "Parts:3310_key_gap"
 			(at 240.03 130.81 0)
 			(effects
@@
 			)
 		)
-		(property "Footprint" "Resistor_SMD:R_0805_2012Metric"
+		(property "Footprint" "Resistor_SMD:R_0402_1005Metric"
 			(at 103.632 166.37 90)
 			(effects
@@
 			)
 		)
-		(property "Footprint" "Resistor_SMD:R_0805_2012Metric"
+		(property "Footprint" "Resistor_SMD:R_0402_1005Metric"
 			(at 36.068 107.95 90)
 			(effects
@@
 			)
 		)
-		(property "Footprint" "Resistor_SMD:R_0805_2012Metric"
+		(property "Footprint" "Resistor_SMD:R_0402_1005Metric"
 			(at 68.072 166.37 90)
 			(effects
@@
 			)
 		)
-		(property "Footprint" "Resistor_SMD:R_0805_2012Metric"
+		(property "Footprint" "Resistor_SMD:R_0402_1005Metric"
 			(at 264.16 116.332 90)
 			(effects
@@
 			)
 		)
-		(property "Footprint" "Capacitor_SMD:C_0805_2012Metric"
+		(property "Footprint" "Capacitor_SMD:C_0402_1005Metric"
 			(at 221.9452 33.02 0)
 			(effects
@@
 			)
 		)
-		(property "Footprint" "Resistor_SMD:R_0805_2012Metric"
+		(property "Footprint" "Resistor_SMD:R_0402_1005Metric"
 			(at 264.16 136.652 90)
 			(effects
@@
 			)
 		)
-		(property "Footprint" "Resistor_SMD:R_0805_2012Metric"
+		(property "Footprint" "Resistor_SMD:R_0402_1005Metric"
 			(at 112.522 166.37 90)
 			(effects
@@
 			)
 		)
-		(property "Footprint" "Resistor_SMD:R_0805_2012Metric"
+		(property "Footprint" "Resistor_SMD:R_0402_1005Metric"
 			(at 85.852 166.37 90)
 			(effects
@@
 			)
 		)
-		(property "Footprint" "Resistor_SMD:R_0805_2012Metric"
+		(property "Footprint" "Resistor_SMD:R_0402_1005Metric"
 			(at 121.412 166.37 90)
 			(effects
@@
 			)
 		)
-		(property "Footprint" "Resistor_SMD:R_0805_2012Metric"
+		(property "Footprint" "Resistor_SMD:R_0402_1005Metric"
 			(at 70.358 107.95 90)
 			(effects
@@
 			)
 		)
-		(property "Footprint" "Resistor_SMD:R_0805_2012Metric"
+		(property "Footprint" "Resistor_SMD:R_0402_1005Metric"
 			(at 264.16 126.492 90)
 			(effects
@@
 			)
 		)
-		(property "Footprint" "Resistor_SMD:R_0805_2012Metric"
+		(property "Footprint" "Resistor_SMD:R_0402_1005Metric"
 			(at 238.252 52.07 90)
 			(effects
@@
 			)
 		)
-		(property "Footprint" "Capacitor_SMD:C_0805_2012Metric"
+		(property "Footprint" "Capacitor_SMD:C_0402_1005Metric"
 			(at 210.5152 33.02 0)
 			(effects
@@
 			)
 		)
-		(property "Footprint" "Resistor_SMD:R_0805_2012Metric"
+		(property "Footprint" "Resistor_SMD:R_0402_1005Metric"
 			(at 53.848 147.32 90)
 			(effects
@@
 			)
 		)
-		(property "Footprint" "Resistor_SMD:R_0805_2012Metric"
+		(property "Footprint" "Resistor_SMD:R_0402_1005Metric"
 			(at 264.16 106.172 90)
 			(effects
@@
 			)
 		)
-		(property "Footprint" "Resistor_SMD:R_0805_2012Metric"
+		(property "Footprint" "Resistor_SMD:R_0402_1005Metric"
 			(at 44.958 177.8 90)
 			(effects
@@
 			)
 		)
-		(property "Footprint" "Resistor_SMD:R_0805_2012Metric"
+		(property "Footprint" "Resistor_SMD:R_0402_1005Metric"
 			(at 59.182 166.37 90)
 			(effects
@@
 			)
 		)
-		(property "Footprint" "Resistor_SMD:R_0805_2012Metric"
+		(property "Footprint" "Resistor_SMD:R_0402_1005Metric"
 			(at 198.628 121.92 90)
 			(effects

Commit message: more pcb routing
Parts:
- renumbered Q6 to Q4, Q7 to Q5, Q8 to Q6, Q9 to Q7, R17 to R15, R18 to R16, R19 to R17, R20 to R18, R21 to R19, R22 to R20, R23 to R21, R24 to R22, R25 to R23, R26 to R24, R27 to R25, R28 to R26, R29 to R27, R30 to R28, R31 to R29, R32 to R30, R33 to R31, R34 to R32, R35 to R33, R36 to R34, R37 to R35, U5 to U6

Commit message: PN update
Parts:
- C19: MPN (none) -> 810-CGA2B3X7R1H104KB; PN (none) -> 810-CGA2B3X7R1H104KB
- C20: MPN (none) -> 77-VJ0402Y103KCAAC; PN (none) -> 77-VJ0402Y103KCAAC
- J5, J6, J7, LS1, SW10, SW11, SW12, SW13, SW14, SW15, SW16, SW17, SW2, SW3, SW4, SW5, SW6, SW7, SW8, SW9: now not fitted
- Q4, Q5, Q7: MPN (none) -> 771-BSS138P215; PN (none) -> 771-BSS138P215
- Q6: MPN (none) -> 942-IRLML6401TRPBF; PN (none) -> 942-IRLML6401TRPBF
- R15, R17, R20: MPN (none) -> 603-RC0402JR-13100KL; PN (none) -> 603-RC0402JR-13100KL
- R16, R19, R21, R22, R23, R24, R25, R26, R27: MPN (none) -> 667-ERJ-2GEJ560X; PN (none) -> 667-ERJ-2GEJ560X
- R18, R31, R32, R33, R34, R35: MPN (none) -> 652-CR0402JW-473GLF; PN (none) -> 652-CR0402JW-473GLF
- R28: MPN (none) -> 603-AF0402JR-071KL; PN (none) -> 603-AF0402JR-071KL
- R29, R30: MPN (none) -> 660-RK73B1ETTP512J; PN (none) -> 660-RK73B1ETTP512J
