File: pmu.kicad_sch (KiCad schematic)
At the start: 21 parts, among them J4 Battery, Q4 BSS138, Q5 BSS84, SW1 POWER ON, U3 MAX1555, U4 TPS63030DSK

Commit message: pcb update
Parts:
- BT1: footprint (none) -> Parts:ML414H; MPN (none) -> ML414H-IV01E; PN (none) -> ML414H-IV01E
- R11, R12, R13, R14, R15, R16: footprint Inductor_SMD:L_0805_2012Metric -> Resistor_SMD:R_0805_2012Metric
Changed lines of the file:
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@@
 	(title_block
 		(title "Mainboard replacement for Nokia 3310")
-		(date "31-10-2024")
+		(date "2-11-2024")
 		(rev "Rev A")
 		(company "M17 Project")
@@
 			)
 		)
-		(property "Footprint" "Inductor_SMD:L_0805_2012Metric"
+		(property "Footprint" "Resistor_SMD:R_0805_2012Metric"
 			(at 119.888 115.57 90)
 			(effects
@@
 			)
 		)
-		(property "Footprint" "Inductor_SMD:L_0805_2012Metric"
+		(property "Footprint" "Resistor_SMD:R_0805_2012Metric"
 			(at 85.852 115.57 90)
 			(effects
@@
 			)
 		)
-		(property "Footprint" "Inductor_SMD:L_0805_2012Metric"
+		(property "Footprint" "Resistor_SMD:R_0805_2012Metric"
 			(at 141.478 113.03 90)
 			(effects
@@
 			)
 		)
-		(property "Footprint" ""
+		(property "Footprint" "Parts:ML414H"
 			(at 226.06 91.186 90)
 			(effects
@@
 			)
 		)
-		(property "PN" ""
+		(property "PN" "ML414H-IV01E"
 			(at 226.06 92.71 0)
 			(effects
@@
 			)
 		)
-		(property "MPN" ""
+		(property "MPN" "ML414H-IV01E"
 			(at 226.06 92.71 0)
 			(effects
@@
 			)
 		)
-		(property "Footprint" "Inductor_SMD:L_0805_2012Metric"
+		(property "Footprint" "Resistor_SMD:R_0805_2012Metric"
 			(at 110.998 90.17 90)
 			(effects
@@
 			)
 		)
-		(property "Footprint" "Inductor_SMD:L_0805_2012Metric"
+		(property "Footprint" "Resistor_SMD:R_0805_2012Metric"
 			(at 81.28 107.442 90)
 			(effects
@@
 			)
 		)
-		(property "Footprint" "Inductor_SMD:L_0805_2012Metric"
+		(property "Footprint" "Resistor_SMD:R_0805_2012Metric"
 			(at 220.98 82.042 90)
 			(effects

Commit message: more pcb routing
Parts:
- C12, C13: footprint Capacitor_SMD:C_0805_2012Metric -> Capacitor_SMD:C_0402_1005Metric
- R11, R12, R13, R14, R15, R16: footprint Resistor_SMD:R_0805_2012Metric -> Resistor_SMD:R_0402_1005Metric
Changed lines of the file:
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@@
 			)
 		)
-		(property "Footprint" "Resistor_SMD:R_0805_2012Metric"
+		(property "Footprint" "Resistor_SMD:R_0402_1005Metric"
 			(at 119.888 115.57 90)
 			(effects
@@
 			)
 		)
-		(property "Footprint" "Resistor_SMD:R_0805_2012Metric"
+		(property "Footprint" "Resistor_SMD:R_0402_1005Metric"
 			(at 85.852 115.57 90)
 			(effects
@@
 			)
 		)
-		(property "Footprint" "Resistor_SMD:R_0805_2012Metric"
+		(property "Footprint" "Resistor_SMD:R_0402_1005Metric"
 			(at 141.478 113.03 90)
 			(effects
@@
 			)
 		)
-		(property "Footprint" "Capacitor_SMD:C_0805_2012Metric"
+		(property "Footprint" "Capacitor_SMD:C_0402_1005Metric"
 			(at 143.8148 95.25 0)
 			(effects
@@
 			)
 		)
-		(property "Footprint" "Resistor_SMD:R_0805_2012Metric"
+		(property "Footprint" "Resistor_SMD:R_0402_1005Metric"
 			(at 110.998 90.17 90)
 			(effects
@@
 			)
 		)
-		(property "Footprint" "Capacitor_SMD:C_0805_2012Metric"
+		(property "Footprint" "Capacitor_SMD:C_0402_1005Metric"
 			(at 91.7448 111.76 0)
 			(effects
@@
 			)
 		)
-		(property "Footprint" "Resistor_SMD:R_0805_2012Metric"
+		(property "Footprint" "Resistor_SMD:R_0402_1005Metric"
 			(at 81.28 107.442 90)
 			(effects
@@
 			)
 		)
-		(property "Footprint" "Resistor_SMD:R_0805_2012Metric"
+		(property "Footprint" "Resistor_SMD:R_0402_1005Metric"
 			(at 220.98 82.042 90)
 			(effects

Commit message: more pcb routing
Parts:
- removed Q4: BSS138, Package_TO_SOT_SMD:SOT-23, symbol Transistor_FET:BSS138
- removed Q5: BSS84, Package_TO_SOT_SMD:SOT-23, symbol Transistor_FET:BSS84
- removed R13: 100k, Resistor_SMD:R_0402_1005Metric, symbol Device:R
- removed R15: 47k, Resistor_SMD:R_0402_1005Metric, symbol Device:R
- added U4: MAX16054, Package_TO_SOT_SMD:TSOT-23-6, symbol Parts:MAX16054
- SW1: value POWER ON -> POWER ON/OFF
- renumbered R14 to R13, R16 to R14, U4 to U5
Connections:
- net GND: now also SW1.2, SW1.4 (A), U4.2 (GND)
- net at D1.1 (K), D2.1 (K), U5.5 (VIN): now also U4.6 (VCC); no longer SW1.2, SW1.4 (A)
- net at SW1.1, SW1.3 (K): now also U4.1 (IN); no longer U5.6 (EN)
- net PWR_ON renamed PWR_OFF
- net PWR_OFF: now also U4.3 (CLR)
- new net: U4.5 (OUT), U5.6 (EN)
- no-connect marks 2 -> 3
Other:
- moved on the sheet: BT1, C13, C14, C15, D3, L1, R13, R14, SW1, U5

Commit message: PN update
Parts:
- C12, C13: MPN (none) -> 810-CGA2B3X7R1H104KB; PN (none) -> 810-CGA2B3X7R1H104KB
- J4: now not fitted
- R11, R12: MPN (none) -> 652-CR0402JW-473GLF; PN (none) -> 652-CR0402JW-473GLF
- R13: MPN (none) -> 603-RC0402JR-13100KL; PN (none) -> 603-RC0402JR-13100KL
- R14: MPN (none) -> 603-AF0402JR-071KL; PN (none) -> 603-AF0402JR-071KL
- U5: MPN (none) -> 595-TPS63030DSKR; PN (none) -> 595-TPS63030DSKR
Changed lines of the file:
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@@
 			)
 		)
-		(property "PN" ""
+		(property "PN" "603-RC0402JR-13100KL"
 			(at 140.97 118.11 0)
 			(effects
@@
 			)
 		)
-		(property "MPN" ""
+		(property "MPN" "603-RC0402JR-13100KL"
 			(at 140.97 118.11 0)
 			(effects
@@
 			)
 		)
-		(property "PN" ""
+		(property "PN" "652-CR0402JW-473GLF"
 			(at 87.63 115.57 0)
 			(effects
@@
 			)
 		)
-		(property "MPN" ""
+		(property "MPN" "652-CR0402JW-473GLF"
 			(at 87.63 115.57 0)
 			(effects
@@
 			)
 		)
+		(property "MPN" "595-TPS63030DSKR"
+			(at 170.18 93.98 0)
+			(effects
+				(font
+					(size 1.27 1.27)
+				)
+				(hide yes)
+			)
+		)
+		(property "PN" "595-TPS63030DSKR"
+			(at 170.18 93.98 0)
+			(effects
+				(font
+					(size 1.27 1.27)
+				)
+				(hide yes)
+			)
+		)
 		(pin "6"
 		)
@@
 		(in_bom yes)
 		(on_board yes)
-		(dnp no)
+		(dnp yes)
 		(property "Reference" "J4"
 			(at 54.61 114.046 0)
@@
 		)
 		(property "Description" "Unpolarized capacitor"
+			(at 147.32 99.06 0)
+			(effects
+				(font
+					(size 1.27 1.27)
+				)
+				(hide yes)
+			)
+		)
+		(property "MPN" "810-CGA2B3X7R1H104KB"
+			(at 147.32 99.06 0)
+			(effects
+				(font
+					(size 1.27 1.27)
+				)
+				(hide yes)
+			)
+		)
+		(property "PN" "810-CGA2B3X7R1H104KB"
 			(at 147.32 99.06 0)
 			(effects
@@
 			)
 		)
+		(property "MPN" "810-CGA2B3X7R1H104KB"
+			(at 92.71 115.57 0)
+			(effects
+				(font
+					(size 1.27 1.27)
+				)
+				(hide yes)
+			)
+		)
+		(property "PN" "810-CGA2B3X7R1H104KB"
+			(at 92.71 115.57 0)
+			(effects
+				(font
+					(size 1.27 1.27)
+				)
+				(hide yes)
+			)
+		)
 		(pin "1"
 		)
@@
 			)
 		)
-		(property "PN" ""
+		(property "PN" "652-CR0402JW-473GLF"
 			(at 81.28 109.22 0)
 			(effects
@@
 			)
 		)
-		(property "MPN" ""
+		(property "MPN" "652-CR0402JW-473GLF"
 			(at 81.28 109.22 0)
 			(effects
@@
 			)
 		)
-		(property "PN" ""
+		(property "PN" "603-AF0402JR-071KL"
 			(at 223.52 83.82 0)
 			(effects
@@
 			)
 		)
-		(property "MPN" ""
+		(property "MPN" "603-AF0402JR-071KL"
 			(at 223.52 83.82 0)
 			(effects
