File: rf.kicad_sch (KiCad schematic)
At the start: 12 parts, among them J2 ANT_A, J3 ANT_B, Q1 BSS138, Q2 IRLML6401, Q3 BSS138, U2 SA868

Commit message: pcb update
Parts:
- R10, R7, R8, R9: footprint Inductor_SMD:L_0805_2012Metric -> Resistor_SMD:R_0805_2012Metric
Changed lines of the file:
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@@
 	(title_block
 		(title "Mainboard replacement for Nokia 3310")
-		(date "31-10-2024")
+		(date "2-11-2024")
 		(rev "Rev A")
 		(company "M17 Project")
@@
 			)
 		)
-		(property "Footprint" "Inductor_SMD:L_0805_2012Metric"
+		(property "Footprint" "Resistor_SMD:R_0805_2012Metric"
 			(at 146.05 75.692 90)
 			(effects
@@
 			)
 		)
-		(property "Footprint" "Inductor_SMD:L_0805_2012Metric"
+		(property "Footprint" "Resistor_SMD:R_0805_2012Metric"
 			(at 173.228 116.84 90)
 			(effects
@@
 			)
 		)
-		(property "Footprint" "Inductor_SMD:L_0805_2012Metric"
+		(property "Footprint" "Resistor_SMD:R_0805_2012Metric"
 			(at 142.748 116.84 90)
 			(effects
@@
 			)
 		)
-		(property "Footprint" "Inductor_SMD:L_0805_2012Metric"
+		(property "Footprint" "Resistor_SMD:R_0805_2012Metric"
 			(at 146.05 98.552 90)
 			(effects

Commit message: more pcb routing
Parts:
- R10, R7, R8, R9: footprint Resistor_SMD:R_0805_2012Metric -> Resistor_SMD:R_0402_1005Metric
Changed lines of the file:
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@@
+		)
+	)
+	(netclass_flag ""
+		(length 2.54)
+		(shape round)
+		(at 193.04 92.71 0)
+		(fields_autoplaced yes)
+		(effects
+			(font
+				(size 1.27 1.27)
+			)
+			(justify left bottom)
+		)
+		(property "Netclass" "RF"
+			(at 193.7385 90.17 0)
+			(effects
+				(font
+					(size 1.27 1.27)
+					(italic yes)
+				)
+				(justify left)
+			)
+		)
+	)
+	(netclass_flag ""
+		(length 2.54)
+		(shape round)
+		(at 157.48 92.71 0)
+		(fields_autoplaced yes)
+		(effects
+			(font
+				(size 1.27 1.27)
+			)
+			(justify left bottom)
+		)
+		(property "Netclass" "RF"
+			(at 158.1785 90.17 0)
+			(effects
+				(font
+					(size 1.27 1.27)
+					(italic yes)
+				)
+				(justify left)
+			)
+		)
+	)
+	(netclass_flag ""
+		(length 2.54)
+		(shape round)
+		(at 129.54 77.47 0)
+		(fields_autoplaced yes)
+		(effects
+			(font
+				(size 1.27 1.27)
+			)
+			(justify left bottom)
+		)
+		(property "Netclass" "Supply"
+			(at 130.2385 74.93 0)
+			(effects
+				(font
+					(size 1.27 1.27)
+					(italic yes)
+				)
+				(justify left)
+			)
 		)
 	)
@@
 			)
 		)
-		(property "Footprint" "Resistor_SMD:R_0805_2012Metric"
+		(property "Footprint" "Resistor_SMD:R_0402_1005Metric"
 			(at 146.05 75.692 90)
 			(effects
@@
 			)
 		)
-		(property "Footprint" "Resistor_SMD:R_0805_2012Metric"
+		(property "Footprint" "Resistor_SMD:R_0402_1005Metric"
 			(at 173.228 116.84 90)
 			(effects
@@
 			)
 		)
-		(property "Footprint" "Resistor_SMD:R_0805_2012Metric"
+		(property "Footprint" "Resistor_SMD:R_0402_1005Metric"
 			(at 142.748 116.84 90)
 			(effects
@@
 			)
 		)
-		(property "Footprint" "Resistor_SMD:R_0805_2012Metric"
+		(property "Footprint" "Resistor_SMD:R_0402_1005Metric"
 			(at 146.05 98.552 90)
 			(effects

Commit message: PN update
Parts:
- J2, J3, U2: now not fitted
- Q1, Q3: MPN (none) -> 771-BSS138P215; PN (none) -> 771-BSS138P215
- Q2: MPN (none) -> 942-IRLML6401TRPBF; PN (none) -> 942-IRLML6401TRPBF
- R10, R7, R8: MPN (none) -> 603-RC0402JR-13100KL; PN (none) -> 603-RC0402JR-13100KL
- R9: MPN (none) -> 652-CR0402JW-473GLF; PN (none) -> 652-CR0402JW-473GLF
Changed lines of the file:
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@@
 		(in_bom yes)
 		(on_board yes)
-		(dnp no)
+		(dnp yes)
 		(fields_autoplaced yes)
 		(property "Reference" "J2"
@@
 			)
 		)
-		(property "PN" ""
+		(property "PN" "603-RC0402JR-13100KL"
 			(at 146.05 77.47 0)
 			(effects
@@
 			)
 		)
-		(property "MPN" ""
+		(property "MPN" "603-RC0402JR-13100KL"
 			(at 146.05 77.47 0)
 			(effects
@@
 		(in_bom yes)
 		(on_board yes)
-		(dnp no)
+		(dnp yes)
 		(fields_autoplaced yes)
 		(property "Reference" "J3"
@@
 			)
 		)
-		(property "PN" ""
+		(property "PN" "603-RC0402JR-13100KL"
 			(at 171.45 116.84 0)
 			(effects
@@
 			)
 		)
-		(property "MPN" ""
+		(property "MPN" "603-RC0402JR-13100KL"
 			(at 171.45 116.84 0)
 			(effects
@@
 			)
 		)
+		(property "MPN" "942-IRLML6401TRPBF"
+			(at 142.24 83.82 0)
+			(effects
+				(font
+					(size 1.27 1.27)
+				)
+				(hide yes)
+			)
+		)
+		(property "PN" "942-IRLML6401TRPBF"
+			(at 142.24 83.82 0)
+			(effects
+				(font
+					(size 1.27 1.27)
+				)
+				(hide yes)
+			)
+		)
 		(pin "1"
 		)
@@
 		(in_bom yes)
 		(on_board yes)
-		(dnp no)
+		(dnp yes)
 		(fields_autoplaced yes)
 		(property "Reference" "U2"
@@
 			)
 		)
-		(property "PN" ""
+		(property "PN" "603-RC0402JR-13100KL"
 			(at 140.97 116.84 0)
 			(effects
@@
 			)
 		)
-		(property "MPN" ""
+		(property "MPN" "603-RC0402JR-13100KL"
 			(at 140.97 116.84 0)
 			(effects
@@
 			)
 		)
-		(property "PN" ""
+		(property "PN" "652-CR0402JW-473GLF"
 			(at 146.05 100.33 0)
 			(effects
@@
 			)
 		)
-		(property "MPN" ""
+		(property "MPN" "652-CR0402JW-473GLF"
 			(at 146.05 100.33 0)
 			(effects
@@
 			)
 		)
+		(property "MPN" "771-BSS138P215"
+			(at 165.1 111.76 0)
+			(effects
+				(font
+					(size 1.27 1.27)
+				)
+				(hide yes)
+			)
+		)
+		(property "PN" "771-BSS138P215"
+			(at 165.1 111.76 0)
+			(effects
+				(font
+					(size 1.27 1.27)
+				)
+				(hide yes)
+			)
+		)
 		(pin "1"
 		)
@@
 			(at 134.62 111.76 0)
 			(effects
+				(font
+					(size 1.27 1.27)
+				)
+				(hide yes)
+			)
+		)
+		(property "MPN" "771-BSS138P215"
+			(at 134.62 111.76 0)
+			(effects
+				(font
+					(size 1.27 1.27)
+				)
+				(hide yes)
+			)
+		)
+		(property "PN" "771-BSS138P215"
+			(at 134.62 111.76 0)
+			(effects
